File: hasp-balloon/electronics/power/power.kicad_sch (KiCad schematic)
At the start: 0 parts

Commit message: feat: schematic v1
Parts:
- added C1, C11, C13, C14, C15, C16, C17, C18, C22, C25, C26, C27, C28, C29, C30, C31, C32, C33, C34, C35, C36, C7, C8, C9: 0.1uF, Capacitor_SMD:C_0805_2012Metric, symbol Device:C
- added C10, C23, C3: 1uF, Capacitor_SMD:C_0603_1608Metric, symbol Device:C
- added C12, C24: 68uF, Capacitor_SMD:C_1206_3216Metric, symbol Device:C
- added C19, C2: 10nF, Capacitor_SMD:C_0603_1608Metric, symbol Device:C
- added C20, C4: 4.7uF, Capacitor_SMD:C_0603_1608Metric, symbol Device:C
- added C21, C6: 10pF, Capacitor_SMD:C_0805_2012Metric, symbol Device:C
- added C5: 0.1UF, Capacitor_SMD:C_0603_1608Metric, symbol Device:C
- added D1, D3: GREEN, LED_SMD:LED_0603_1608Metric, symbol Device:LED
- added FB1, FB2, FB3, FB4, FB5, FB6, FB7, FB8: FerriteBead_Small, symbol Device:FerriteBead_Small
- added J1, J10, J11, J2, J7, J9: Molex Pico-Lock, symbol Connector_Generic:Conn_01x02
- added J12, J13, J14, J15, J16, J17, J3, J5: Wire-to-Board, Connector_PinHeader_2.54mm:PinHeader_1x02_P2.54mm_Vertical, symbol Connector_Generic:Conn_01x02
- added J4, J6: Molex Pico-Lock, symbol Connector_Generic:Conn_01x04
- added J8: DB9, symbol Connector:DE9_Socket
- added L1, L3: 10uH, Inductor_SMD:L_Coilcraft_XxL4040, symbol Device:L
- added M1, M2, M3: Servo (Pico-Lock), symbol Motor:Motor_Servo
- added R1, R9: 110k, Resistor_SMD:R_0603_1608Metric, symbol Device:R
- added R10, R14, R15: 10k, Resistor_SMD:R_0805_2012Metric, symbol Device:R
- added R11: 114k, Resistor_SMD:R_0805_2012Metric, symbol Device:R
- added R12, R7: 150, Resistor_SMD:R_0805_2012Metric, symbol Device:R
- added R13, R19, R20, R21, R22, R23, R24, R25: 400, Resistor_SMD:R_0603_1608Metric, symbol Device:R
- added R16: 2m, Resistor_SMD:R_2512_6332Metric, symbol Device:R
- added R17, R18: 10, Resistor_SMD:R_0603_1608Metric, symbol Device:R
- added R2, R4, R6, R8: 50k, Resistor_SMD:R_0603_1608Metric, symbol Device:R
- added R3: 243k, Resistor_SMD:R_0805_2012Metric, symbol Device:R
- added R39: 12.5, Resistor_SMD:R_0603_1608Metric, symbol Device:R
- added R5: 1M, Resistor_SMD:R_0805_2012Metric, symbol Device:R
- added TP1, TP3: ~, TestPoint:TestPoint_Keystone_5000-5004_Miniature, symbol Connector:TestPoint
- added U1: RASPBERRY_PI_ZERO_2_W, RASPBERRY_PI_ZERO_2_W:MODULE_RASPBERRY_PI_ZERO_2_W, symbol RASPBERRY_PI_ZERO_2_W:RASPBERRY_PI_ZERO_2_W
- added U10, U12, U16, U4, U9: TPS281C30, Package_DFN_QFN:Texas_RGW0020A_VQFN-20-1EP_5x5mm_P0.65mm_EP3.15x3.15mm_ThermalVias, symbol pdu:TPS281C30
- added U11: MCP3201, Package_SO:SOIC-8-1EP_3.9x4.9mm_P1.27mm_EP2.41x3.81mm, symbol Analog_ADC:MCP3201
- added U13: MAX3110E, symbol hasp:MAX3110E
- added U14: INA219AxD, Package_SO:SOIC-8_3.9x4.9mm_P1.27mm, symbol Sensor_Energy:INA219AxD
- added U15, U17, U18, U19, U20, U21, U22, U7: MAX31865, Package_SO:SSOP-20_5.3x7.2mm_P0.65mm, symbol Sensor_Temperature:MAX31865xAP
- added U2: TMP36FSZ, Package_SO:SOIC-8-1EP_3.9x4.9mm_P1.27mm_EP2.41x3.3mm, symbol pdu:TMP36FSZ
- added U3, U6: LT8610, Package_SO:MSOP-16-1EP_3x4.039mm_P0.5mm_EP1.651x2.845mm_ThermalVias, symbol Regulator_Switching:LT8610
- added U5: MAX3232, Package_SO:SOIC-16_3.9x9.9mm_P1.27mm, symbol Interface_UART:MAX3232
- added U8: MS560702BA03-50, MS560702BA03-50:SON125P300X500X100-8N, symbol MS560702BA03-50:MS560702BA03-50
- added Y1: 1.8432 MHz, symbol Device:Crystal
Connections:
- new net: J13.1 (Pin_1), U18.10 (RTDIN+), U18.8 (FORCE+)
- new net: J13.2 (Pin_2), U18.11 (RTDIN-), U18.12 (FORCE-)
- new net: C32.1, FB6.2, U20.3 (VDD)
- new net: J15.1 (Pin_1), U20.10 (RTDIN+), U20.8 (FORCE+)
- new net: J15.2 (Pin_2), U20.11 (RTDIN-), U20.12 (FORCE-)
- new net: R23.1, U20.4 (BIAS), U20.5 (REFIN+)
- new net: R23.2, U20.6 (REFIN-), U20.7 (ISENSOR)
- new net: D1.1 (K), R7.2
- new net: C36.1, FB8.2, U22.3 (VDD)
- new net: C23.1, U6.13 (INTVcc)
- new net: R13.1, U7.4 (BIAS), U7.5 (REFIN+)
- new net: R13.2, U7.6 (REFIN-), U7.7 (ISENSOR)
- new net: J3.1 (Pin_1), U15.10 (RTDIN+), U15.8 (FORCE+)
- new net: J3.2 (Pin_2), U15.11 (RTDIN-), U15.12 (FORCE-)
- new net: C9.1, FB2.2, U15.3 (VDD)
- new net: R19.1, U15.4 (BIAS), U15.5 (REFIN+)
- new net: R19.2, U15.6 (REFIN-), U15.7 (ISENSOR)
- new net: C22.1, U6.12 (BST)
- new net: C30.1, FB5.2, U19.3 (VDD)
- new net: C3.1, R17.2, U14.8 (IN+)
- new net: C3.2, R18.2, U14.7 (IN-)
- new net: C16.1, U5.4 (C2+)
- new net: C16.2, U5.5 (C2-)
- new net: C34.1, FB7.2, U21.3 (VDD)
- new net: R2.1, U4.1 (ILIM)
- new net: C17.2, U5.2 (VS+)
- new net: R20.1, U17.4 (BIAS), U17.5 (REFIN+)
- new net: R20.2, U17.6 (REFIN-), U17.7 (ISENSOR)
- new net: R21.1, U18.4 (BIAS), U18.5 (REFIN+)
- new net: R21.2, U18.6 (REFIN-), U18.7 (ISENSOR)
- new net: J12.1 (Pin_1), U17.10 (RTDIN+), U17.8 (FORCE+)
- new net: J12.2 (Pin_2), U17.11 (RTDIN-), U17.12 (FORCE-)
- new net: C15.1, U5.3 (C1-)
- new net: C15.2, U5.1 (C1+)
- new net: C8.1, U3.12 (BST)
- new net: C10.1, U3.13 (INTVcc)
- new net: C2.2, U3.2 (TR/SS)
- new net: R1.1, U3.3 (RT)
- new net: C26.1, FB1.2, U7.3 (VDD)
- new net: R9.1, U6.3 (RT)
- new net: C28.1, FB4.2, U18.3 (VDD)
- new net: D3.1 (K), R12.2
- new net: U13. (DIN), Y1.1
- new net: U13. (DIN), Y1.2
- new net: C19.2, U6.2 (TR/SS)
- new net: R25.1, U22.4 (BIAS), U22.5 (REFIN+)
- new net: R25.2, U22.6 (REFIN-), U22.7 (ISENSOR)
- new net: R39.1, U16.1 (ILIM)
- new net: R6.1, U10.1 (ILIM)
- new net: J17.1 (Pin_1), U22.10 (RTDIN+), U22.8 (FORCE+)
- new net: J17.2 (Pin_2), U22.11 (RTDIN-), U22.12 (FORCE-)
- new net: J16.1 (Pin_1), U21.10 (RTDIN+), U21.8 (FORCE+)
- new net: J16.2 (Pin_2), U21.11 (RTDIN-), U21.12 (FORCE-)
- new net: J5.1 (Pin_1), U7.10 (RTDIN+), U7.8 (FORCE+)
- new net: J5.2 (Pin_2), U7.11 (RTDIN-), U7.12 (FORCE-)
- new net: R8.1, U12.1 (ILIM)
- new net: R4.1, U9.1 (ILIM)
- new net: C13.1, FB3.2, U17.3 (VDD)
- new net: C18.2, U5.6 (VS-)
- new net: R24.1, U21.4 (BIAS), U21.5 (REFIN+)
- new net: R24.2, U21.6 (REFIN-), U21.7 (ISENSOR)
- new net: R22.1, U19.4 (BIAS), U19.5 (REFIN+)
- new net: R22.2, U19.6 (REFIN-), U19.7 (ISENSOR)
- new net: J14.1 (Pin_1), U19.10 (RTDIN+), U19.8 (FORCE+)
- new net: J14.2 (Pin_2), U19.11 (RTDIN-), U19.12 (FORCE-)
- new net 12V: C20.1, C21.2, C24.2, C4.1, D3.2 (A), J2.1 (Pin_1), L3.2, R11.2, R16.2, R17.1, TP3.1, U10.10 (VS), U10.11 (VS), U10.12 (VS), U10.13 (VS), U12.10 (VS), U12.11 (VS), U12.12 (VS), U12.13 (VS), U16.10 (VS), U16.11 (VS), U16.12 (VS), U16.13 (VS), U3.4 (EN/UV), U3.5 (VIN), U3.6 (VIN), U4.10 (VS), U4.11 (VS), U4.12 (VS), U4.13 (VS), U6.14 (BIAS), U6.4 (EN/UV), U6.5 (VIN), U6.6 (VIN), U9.10 (VS), U9.11 (VS), U9.12 (VS), U9.13 (VS)
- new net 12V_STAT: U1.11 (GPIO17/GPIO_GEN0), U6.15 (PG)
- new net 28V_CS: J7.1 (Pin_1), R16.1, R18.1
- new net 3V3: C1.2, C11.2, C14.2, C25.2, C27.2, C29.2, C31.2, C33.2, C35.2, C5.2, C7.2, FB1.1, FB2.1, FB3.1, FB4.1, FB5.1, FB6.1, FB7.1, FB8.1, R14.2, R15.2, U1.1 (3V3_1), U1.17 (3V3_17), U14.5 (VS), U15.2 (DVDD), U17.2 (DVDD), U18.2 (DVDD), U19.2 (DVDD), U2.5 (SHUTDOWN), U2.8 (V_IN), U20.2 (DVDD), U21.2 (DVDD), U22.2 (DVDD), U5.16 (VCC), U7.2 (DVDD), U8.1 (VDD)
- new net 5V: C12.2, C6.2, D1.2 (A), J4.1 (Pin_1), L1.2, M1.2 (+), M2.2 (+), M3.2 (+), R5.2, TP1.1, U1.2 (5V_2), U1.4 (5V_4), U11.1 (Vref), U11.8 (Vdd), U13. (DIN), U3.14 (BIAS)
- new net 5V_STAT: U1.12 (GPIO18/GPIO_GEN1), U3.15 (PG)
- new net ANALOG_TEMP: U11.2 (IN+), U2.1 (V_OUT)
- new net FB_3: C21.1, C6.1, R10.2, R11.1, R3.2, R5.1, U3.16 (FB), U6.16 (FB)
- new net GND: C1.1, C10.2, C11.1, C12.1, C13.2, C14.1, C17.1, C18.1, C19.1, C2.1, C20.2, C23.2, C24.1, C25.1, C26.2, C27.1, C28.2, C29.1, C30.2, C31.1, C32.2, C33.1, C34.2, C35.1, C36.2, C4.2, C5.1, C7.1, C9.2, J1.2 (Pin_2), J10.2 (Pin_2), J11.2 (Pin_2), J2.2 (Pin_2), J4.4 (Pin_4), J6.4 (Pin_4), J7.2 (Pin_2), J8.5, J9.2 (Pin_2), M1.3 (-), M2.3 (-), M3.3 (-), R1.2, R10.1, R12.1, R2.2, R3.1, R39.2, R4.2, R6.2, R7.1, R8.2, R9.2, U1.14 (GND_14), U1.20 (GND_20), U1.25 (GND_25), U1.30 (GND_30), U1.34 (GND_34), U1.39 (GND_39), U1.6 (GND_6), U1.9 (GND_9), U10.18 (GND), U11.3 (IN-), U11.4 (Vss), U12.18 (GND), U13. (DIN), U14.1 (A1), U14.6 (GND), U15.13 (GND), U15.18 (DGND), U15.19 (GND), U15.9 (FORCE2), U16.18 (GND), U17.13 (GND), U17.18 (DGND), U17.19 (GND), U17.9 (FORCE2), U18.13 (GND), U18.18 (DGND), U18.19 (GND), U18.9 (FORCE2), U19.13 (GND), U19.18 (DGND), U19.19 (GND), U19.9 (FORCE2), U2.4 (GND), U20.13 (GND), U20.18 (DGND), U20.19 (GND), U20.9 (FORCE2), U21.13 (GND), U21.18 (DGND), U21.19 (GND), U21.9 (FORCE2), U22.13 (GND), U22.18 (DGND), U22.19 (GND), U22.9 (FORCE2), U3.17 (GND), U3.7 (GND), U3.8 (GND), U4.18 (GND), U5.15 (GND), U6.17 (GND), U6.7 (GND), U6.8 (GND), U7.13 (GND), U7.18 (DGND), U7.19 (GND), U7.9 (FORCE2), U8.3 (GND), U9.18 (GND)
- new net HEAT_1_EN: U4.15 (EN)
- new net HEAT_1_PWR: J1.1 (Pin_1), U4.3 (VOUT), U4.4 (VOUT), U4.5 (VOUT), U4.6 (VOUT)
- new net HEAT_2_EN: U1.15 (GPIO22/GPIO_GEN3), U9.15 (EN)
- new net HEAT_2_PWR: J9.1 (Pin_1), U9.3 (VOUT), U9.4 (VOUT), U9.5 (VOUT), U9.6 (VOUT)
- new net HEAT_3_EN: U1.16 (GPIO23/GPIO_GEN4), U10.15 (EN)
- new net HEAT_3_PWR: J10.1 (Pin_1), U10.3 (VOUT), U10.4 (VOUT), U10.5 (VOUT), U10.6 (VOUT)
- new net HEAT_4_EN: U1.18 (GPIO24/GPIO_GEN5), U12.15 (EN)
- new net HEAT_4_PWR: J11.1 (Pin_1), U12.3 (VOUT), U12.4 (VOUT), U12.5 (VOUT), U12.6 (VOUT)
- new net MISO: U1.21 (GPIO9/SPI_MISO), U11.6 (Dout), U13. (DIN), U15.17 (SDO), U17.17 (SDO), U18.17 (SDO), U19.17 (SDO), U20.17 (SDO), U21.17 (SDO), U22.17 (SDO), U7.17 (SDO)
- new net MOSI: U1.19 (GPIO10/SPI_MOSI), U13. (DIN), U15.14 (SDI), U17.14 (SDI), U18.14 (SDI), U19.14 (SDI), U20.14 (SDI), U21.14 (SDI), U22.14 (SDI), U7.14 (SDI)
- new net POPS_CS: U13. (DIN)
- new net PUMP_PWR: U16.3 (VOUT), U16.4 (VOUT), U16.5 (VOUT), U16.6 (VOUT)
- new net PUMP_PWR_EN: U1.7 (GPIO4/GPIO_GCLK), U16.15 (EN)
- new net R1IN: J8.3, J8.7, U13. (DIN)
- new net R1OUT: U13. (DIN)
- new net R2IN: U13. (DIN)
- new net R2OUT: U13. (DIN)
- new net RS232_RX: J6.2 (Pin_2), U5.13 (R1IN)
- new net RS232_TX: J6.1 (Pin_1), U5.14 (T1OUT)
- new net RTD1_CS: U1.29 (GPIO5), U7.16 (~{CS})
- new net RTD2_CS: U1.31 (GPIO6), U15.16 (~{CS})
- new net RTD3_CS: U1.26 (GPIO7/SPI_~{CE1}), U17.16 (~{CS})
- new net RTD4_CS: U18.16 (~{CS})
- new net RTD5_CS: U19.16 (~{CS})
- new net RTD6_CS: U20.16 (~{CS})
- new net RTD7_CS: U21.16 (~{CS})
- new net RTD8_CS: U22.16 (~{CS})
- new net SCL: J4.2 (Pin_2), R15.1, U1.5 (GPIO3/SCL), U14.4 (SCL), U8.8 (SCLK)
- new net SCLK: U1.23 (GPIO11/SPI_SCLK), U11.7 (CLK), U13. (DIN), U15.15 (SCLK), U17.15 (SCLK), U18.15 (SCLK), U19.15 (SCLK), U20.15 (SCLK), U21.15 (SCLK), U22.15 (SCLK), U7.15 (SCLK)
- new net SDA: J4.3 (Pin_3), R14.1, U1.3 (GPIO2/SDA1), U14.2 (A0), U14.3 (SDA), U8.7 (SDI/SDA)
- new net SERVO_1_PWM: M1.1 (PWM)
- new net SERVO_2_PWM: M2.1 (PWM)
- new net SERVO_3_PWM: M3.1 (PWM)
- new net SW_3: C22.2, C8.2, L1.1, L3.1, U3.10 (SW), U3.11 (SW), U3.9 (SW), U6.10 (SW), U6.11 (SW), U6.9 (SW)
- new net T1IN: U13. (DIN)
- new net T1OUT: J8.8, U13. (DIN)
- new net T2IN: U13. (DIN)
- new net T2OUT: J8.2, U13. (DIN)
- new net TEMP_CS: U1.24 (GPIO8/SPI_~{CE0}), U11.5 (~{CS}/SHDN)
- new net UART_RX: U1.10 (GPIO15/RXD0), U5.12 (R1OUT)
- new net UART_TX: U1.8 (GPIO14/TXD0), U5.11 (T1IN)
- new net VAC_EN: U1.40 (GPIO21)
- new net ~{PUMP_PWR_FAULT}: U1.32 (GPIO12), U16.17 (~{FAULT})
- no-connect marks 0 -> 52
Other:
- note added: "12.5 = 4A Limit"
- note added: "1206"
- note added: "12V Regulator"
- note added: "2512 (7W)"
- note added: "50k = 1A Limit"
- note added: "5V Regulator"
- note added: "ALL PASSIVES ARE 0805 UNLESS OTHERWISE SPECIFIED"
- note added: "Board Temperature Sensor"
- note added: "Flow Meter Connector"
- note added: "HASP Interface"
- note added: "Heater Drivers"
- note added: "I2C Address: 0x42"
- note added: "I2C Pullups"
- note added: "POPS Connectors"
- note added: "Payload Computer"
- note added: "Power Monitor"
- note added: "Pressure Sensor"
- note added: "RS-232 to SPI (POPS)"
- note added: "RS232 Level Shifter (HASP)"
- note added: "RTD Temperature Sensors"
- note added: "Servo Cap Control"
- note added: "Vacuum Pump Load Driver"
- note added: "Voltage Regulators"
- company: (none) -> UChicago Space Program
- title: (none) -> PASCAL Avionics Card
